Commit message: Add Gazebo plugins and warehouse simulation for the AMR

File: amr_description/urdf/amr.urdf.xacro (robot description, xacro)
@@ -7,4 +7,11 @@
   <xacro:property name="base_mass" value="15.0"/>
   <xacro:property name="ground_clearance" value="0.03"/>
+  <xacro:property name="wheel_radius" value="0.08"/>
+  <xacro:property name="wheel_width" value="0.05"/>
+  <xacro:property name="wheel_mass" value="1.0"/>
+  <xacro:property name="caster_radius" value="0.03"/>
+  <xacro:property name="caster_x" value="0.22"/>
+  <!-- Height of base_link (centre of the box) above the ground -->
+  <xacro:property name="base_z" value="${ground_clearance + base_height / 2}"/>
   <!-- ========== Footprint: on the ground, under the robot centre ========== -->
   <link name="base_footprint"/>
@@ -31,9 +38,170 @@
     </inertial>
   </link>
-  <!-- base_link sits at the centre of the box: clearance + half the height -->
   <joint name="base_joint" type="fixed">
     <parent link="base_footprint"/>
     <child link="base_link"/>
-    <origin xyz="0 0 ${ground_clearance + base_height / 2}" rpy="0 0 0"/>
+    <origin xyz="0 0 ${base_z}" rpy="0 0 0"/>
   </joint>
+  <!-- ========== Drive wheel macro: side = 1 (left) or -1 (right) ========== -->
+  <xacro:macro name="drive_wheel" params="name side">
+    <link name="${name}_wheel">
+      <visual>
+        <!-- a cylinder points along Z; roll it 90 deg so it points along Y -->
+        <origin xyz="0 0 0" rpy="${pi / 2} 0 0"/>
+        <geometry>
+          <cylinder radius="${wheel_radius}" length="${wheel_width}"/>
+        </geometry>
+        <material name="black">
+          <color rgba="0.1 0.1 0.1 1.0"/>
+        </material>
+      </visual>
+      <collision>
+        <origin xyz="0 0 0" rpy="${pi / 2} 0 0"/>
+        <geometry>
+          <cylinder radius="${wheel_radius}" length="${wheel_width}"/>
+        </geometry>
+      </collision>
+      <inertial>
+        <origin xyz="0 0 0" rpy="${pi / 2} 0 0"/>
+        <mass value="${wheel_mass}"/>
+        <inertia ixx="${wheel_mass / 12.0 * (3 * wheel_radius**2 + wheel_width**2)}"
+                 ixy="0" ixz="0"
+                 iyy="${wheel_mass / 12.0 * (3 * wheel_radius**2 + wheel_width**2)}"
+                 iyz="0" izz="${wheel_mass / 2.0 * wheel_radius**2}"/>
+      </inertial>
+    </link>
+    <joint name="${name}_wheel_joint" type="continuous">
+      <parent link="base_link"/>
+      <child link="${name}_wheel"/>
+      <!-- middle of the side, just outside the box, axle at wheel_radius above the ground -->
+      <origin xyz="0 ${side * (base_width / 2 + wheel_width / 2)} ${wheel_radius - base_z}"
+              rpy="0 0 0"/>
+      <axis xyz="0 1 0"/>
+    </joint>
+  </xacro:macro>
+  <xacro:drive_wheel name="left" side="1"/>
+  <xacro:drive_wheel name="right" side="-1"/>
+  <!-- ========== Caster macro: position = 1 (front) or -1 (rear) ========== -->
+  <xacro:macro name="caster" params="name position">
+    <link name="${name}_caster">
+      <visual>
+        <geometry>
+          <sphere radius="${caster_radius}"/>
+        </geometry>
+        <material name="grey">
+          <color rgba="0.6 0.6 0.6 1.0"/>
+        </material>
+      </visual>
+      <collision>
+        <geometry>
+          <sphere radius="${caster_radius}"/>
+        </geometry>
+      </collision>
+      <inertial>
+        <mass value="0.2"/>
+        <inertia ixx="${0.4 * 0.2 * caster_radius**2}" ixy="0" ixz="0"
+                 iyy="${0.4 * 0.2 * caster_radius**2}" iyz="0"
+                 izz="${0.4 * 0.2 * caster_radius**2}"/>
+      </inertial>
+    </link>
+    <joint name="${name}_caster_joint" type="fixed">
+      <parent link="base_link"/>
+      <child link="${name}_caster"/>
+      <!-- the sphere touches the ground: its centre is caster_radius above it -->
+      <origin xyz="${position * caster_x} 0 ${caster_radius - base_z}" rpy="0 0 0"/>
+    </joint>
+  </xacro:macro>
+  <xacro:caster name="front" position="1"/>
+  <xacro:caster name="rear" position="-1"/>
+  <!-- ========== Cargo deck: plate + low rim, behind the LiDAR ========== -->
+  <xacro:property name="deck_length" value="0.48"/>
+  <xacro:property name="deck_x" value="-0.05"/>        <!-- shifted back to leave room for the LiDAR -->
+  <xacro:property name="plate_thickness" value="0.01"/>
+  <xacro:property name="rim_height" value="0.04"/>
+  <xacro:property name="rim_thickness" value="0.01"/>
+  <link name="cargo_deck">
+    <visual>
+      <origin xyz="0 0 ${plate_thickness / 2}"/>
+      <geometry>
+        <box size="${deck_length} ${base_width} ${plate_thickness}"/>
+      </geometry>
+      <material name="grey"/>
+    </visual>
+    <collision>
+      <origin xyz="0 0 ${plate_thickness / 2}"/>
+      <geometry>
+        <box size="${deck_length} ${base_width} ${plate_thickness}"/>
+      </geometry>
+    </collision>
+    <inertial>
+      <mass value="1.0"/>
+      <inertia ixx="0.01" ixy="0" ixz="0" iyy="0.02" iyz="0" izz="0.03"/>
+    </inertial>
+  </link>
+  <joint name="cargo_deck_joint" type="fixed">
+    <parent link="base_link"/>
+    <child link="cargo_deck"/>
+    <!-- sits on top of the box -->
+    <origin xyz="${deck_x} 0 ${base_height / 2}"/>
+  </joint>
+  <!-- one rim wall: size and position relative to the deck -->
+  <xacro:macro name="rim" params="name sx sy x y">
+    <link name="rim_${name}">
+      <visual>
+        <geometry>
+          <box size="${sx} ${sy} ${rim_height}"/>
+        </geometry>
+        <material name="grey"/>
+      </visual>
+      <collision>
+        <geometry>
+          <box size="${sx} ${sy} ${rim_height}"/>
+        </geometry>
+      </collision>
+      <inertial>
+        <mass value="0.1"/>
+        <inertia ixx="0.001" ixy="0" ixz="0" iyy="0.001" iyz="0" izz="0.001"/>
+      </inertial>
+    </link>
+    <joint name="rim_${name}_joint" type="fixed">
+      <parent link="cargo_deck"/>
+      <child link="rim_${name}"/>
+      <origin xyz="${x} ${y} ${plate_thickness + rim_height / 2}"/>
+    </joint>
+  </xacro:macro>
+  <xacro:rim name="front" sx="${rim_thickness}" sy="${base_width}"
+             x="${deck_length / 2 - rim_thickness / 2}" y="0"/>
+  <xacro:rim name="rear" sx="${rim_thickness}" sy="${base_width}"
+             x="${-deck_length / 2 + rim_thickness / 2}" y="0"/>
+  <xacro:rim name="left" sx="${deck_length}" sy="${rim_thickness}"
+             x="0" y="${base_width / 2 - rim_thickness / 2}"/>
+  <xacro:rim name="right" sx="${deck_length}" sy="${rim_thickness}"
+             x="0" y="${-base_width / 2 + rim_thickness / 2}"/>
+  <!-- ========== LiDAR: on the front of the top, ahead of the cargo deck ========== -->
+  <xacro:property name="lidar_radius" value="0.04"/>
+  <xacro:property name="lidar_height" value="0.05"/>
+  <link name="lidar_link">
+    <visual>
+      <geometry>
+        <cylinder radius="${lidar_radius}" length="${lidar_height}"/>
+      </geometry>
+      <material name="black"/>
+    </visual>
+    <collision>
+      <geometry>
+        <cylinder radius="${lidar_radius}" length="${lidar_height}"/>
+      </geometry>
+    </collision>
+    <inertial>
+      <mass value="0.2"/>
+      <inertia ixx="0.0001" ixy="0" ixz="0" iyy="0.0001" iyz="0" izz="0.0002"/>
+    </inertial>
+  </link>
+  <joint name="lidar_joint" type="fixed">
+    <parent link="base_link"/>
+    <child link="lidar_link"/>
+    <origin xyz="${base_length / 2 - 0.05} 0 ${base_height / 2 + lidar_height / 2}"/>
+  </joint>
+    <!-- Simulation-only parts (friction, DiffDrive, LiDAR sensor) -->
+  <xacro:include filename="amr.gazebo.xacro"/>
 </robot>

Commit message: AMR navigates the warehouse with Nav2: bridge TwistStamped, initial pose, raised LiDAR

File: amr_description/urdf/amr.urdf.xacro (robot description, xacro)
@@ -201,5 +201,5 @@
     <parent link="base_link"/>
     <child link="lidar_link"/>
-    <origin xyz="${base_length / 2 - 0.05} 0 ${base_height / 2 + lidar_height / 2}"/>
+       <origin xyz="${base_length / 2 - 0.05} 0 ${base_height / 2 + plate_thickness + rim_height + lidar_height / 2 + 0.01}"/>
   </joint>
     <!-- Simulation-only parts (friction, DiffDrive, LiDAR sensor) -->

Commit message: Modern trim: dark blue body, cover, LED strip, bumper, red LiDAR

File: amr_description/urdf/amr.urdf.xacro (robot description, xacro)
@@ -34,5 +34,5 @@
       </geometry>
       <material name="mir_grey">
-        <color rgba="0.75 0.75 0.75 1.0"/>
+        <color rgba="0.05 0.15 0.40 1.0"/>
       </material>
     </visual>
@@ -148,6 +148,6 @@
         <mesh filename="${mesh_dir}/sick_lms-100.stl"/>
       </geometry>
-      <material name="sick_yellow">
-        <color rgba="0.95 0.75 0.1 1.0"/>
+            <material name="sick_red">
+        <color rgba="0.85 0.1 0.1 1.0"/>
       </material>
     </visual>
@@ -168,4 +168,47 @@
     <origin xyz="${body_dx + body_length / 2 - 0.08} 0 ${body_top + lidar_mount_height}"/>
   </joint>
+  <!-- ========== Modern trim: visual only, no collision ========== -->
+  <link name="body_trim">
+    <!-- light grey top cover: the cargo surface -->
+    <visual>
+      <origin xyz="${body_dx} 0 ${body_top + 0.004}"/>
+      <geometry>
+        <box size="${body_length - 0.03} ${body_width - 0.03} 0.008"/>
+      </geometry>
+      <material name="cover_grey">
+        <color rgba="0.85 0.87 0.90 1.0"/>
+      </material>
+    </visual>
+    <!-- cyan LED strip all around, just below the top -->
+    <visual>
+      <origin xyz="${body_dx} 0 ${body_top - 0.05}"/>
+      <geometry>
+        <box size="${body_length + 0.006} ${body_width + 0.006} 0.015"/>
+      </geometry>
+      <material name="led_cyan">
+        <color rgba="0.0 0.85 1.0 1.0"/>
+      </material>
+    </visual>
+    <!-- black rubber bumper around the bottom -->
+    <visual>
+      <origin xyz="${body_dx} 0 ${body_bottom + 0.03}"/>
+      <geometry>
+        <box size="${body_length + 0.012} ${body_width + 0.012} 0.06"/>
+      </geometry>
+      <material name="bumper_black">
+        <color rgba="0.05 0.05 0.05 1.0"/>
+      </material>
+    </visual>
+    <!-- a tiny mass, otherwise Gazebo drops the link and its visuals -->
+    <inertial>
+      <mass value="0.1"/>
+      <inertia ixx="0.0001" ixy="0" ixz="0" iyy="0.0001" iyz="0" izz="0.0001"/>
+    </inertial>
+  </link>
+  <joint name="body_trim_joint" type="fixed">
+    <parent link="base_link"/>
+    <child link="body_trim"/>
+    <origin xyz="0 0 0"/>
+  </joint>
   <!-- Simulation-only parts (friction, DiffDrive, LiDAR sensor) -->
   <xacro:include filename="amr.gazebo.xacro"/>

Commit message: Front camera tilted 40 deg down, bridged to ROS

File: amr_description/urdf/amr.urdf.xacro (robot description, xacro)
@@ -211,5 +211,54 @@
     <origin xyz="0 0 0"/>
   </joint>
+  <!-- ========== Downward camera: reads AprilTags on the floor ========== -->
+  <!-- Under the robot, between the drive wheels (the centre of rotation) -->
+  <link name="camera_link">
+    <visual>
+      <geometry>
+        <box size="0.03 0.05 0.03"/>
+      </geometry>
+      <material name="black"/>
+    </visual>
+    <inertial>
+      <mass value="0.05"/>
+      <inertia ixx="0.00001" ixy="0" ixz="0" iyy="0.00001" iyz="0" izz="0.00001"/>
+    </inertial>
+  </link>
+  <!-- pitch +90 deg: the camera's +x (its viewing direction in Gazebo) points down -->
+  <joint name="camera_joint" type="fixed">
+    <parent link="base_link"/>
+    <child link="camera_link"/>
+    <origin xyz="${body_dx + body_length / 2 + 0.015} 0 0.25" rpy="0 ${40 * pi / 180} 0"/>
+  </joint>
+  <!-- ROS camera convention: z out of the lens, x right, y down in the image -->
+  <link name="camera_optical_link"/>
+  <joint name="camera_optical_joint" type="fixed">
+    <parent link="camera_link"/>
+    <child link="camera_optical_link"/>
+    <origin xyz="0 0 0" rpy="${-pi / 2} 0 ${-pi / 2}"/>
+  </joint>
   <!-- Simulation-only parts (friction, DiffDrive, LiDAR sensor) -->
   <xacro:include filename="amr.gazebo.xacro"/>
+  <!-- Downward camera: 640x480 at 15 Hz, wide lens to see the floor tag -->
+  <gazebo reference="camera_link">
+    <sensor name="floor_camera" type="camera">
+      <topic>camera/image</topic>
+      <gz_frame_id>camera_optical_link</gz_frame_id>
+      <update_rate>15</update_rate>
+      <always_on>true</always_on>
+      <visualize>true</visualize>
+      <camera>
+        <horizontal_fov>1.75</horizontal_fov>
+        <image>
+          <width>640</width>
+          <height>480</height>
+          <format>R8G8B8</format>
+        </image>
+        <clip>
+          <near>0.02</near>
+          <far>2.0</far>
+        </clip>
+      </camera>
+    </sensor>
+  </gazebo>
 </robot>
